File: ADC.kicad_sch (KiCad schematic)
At the start: 36 parts, among them U10 ADS1015IDGSR, U11 ADS1015IDGSR

Commit message: Added pots to schem
Parts:
- RV1, RV2, RV3, RV4, RV5, RV6, RV7, RV8: footprint (none) -> TeenieWeenieLibrary:POT_PTV09A-4025U-B104
Changed lines of the file:
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@@
       (effects (font (size 1.27 1.27)) (justify right) hide)
     )
-    (property "Footprint" "" (at 60.96 74.93 0)
+    (property "Footprint" "TeenieWeenieLibrary:POT_PTV09A-4025U-B104" (at 60.96 74.93 0)
       (effects (font (size 1.27 1.27)) hide)
     )
@@
       (effects (font (size 1.27 1.27)) (justify right) hide)
     )
-    (property "Footprint" "" (at 60.96 113.03 0)
+    (property "Footprint" "TeenieWeenieLibrary:POT_PTV09A-4025U-B104" (at 60.96 113.03 0)
       (effects (font (size 1.27 1.27)) hide)
     )
@@
       (effects (font (size 1.27 1.27)) (justify right) hide)
     )
-    (property "Footprint" "" (at 41.91 74.93 0)
+    (property "Footprint" "TeenieWeenieLibrary:POT_PTV09A-4025U-B104" (at 41.91 74.93 0)
       (effects (font (size 1.27 1.27)) hide)
     )
@@
       (effects (font (size 1.27 1.27)) (justify right) hide)
     )
-    (property "Footprint" "" (at 22.86 113.03 0)
+    (property "Footprint" "TeenieWeenieLibrary:POT_PTV09A-4025U-B104" (at 22.86 113.03 0)
       (effects (font (size 1.27 1.27)) hide)
     )
@@
       (effects (font (size 1.27 1.27)) (justify right) hide)
     )
-    (property "Footprint" "" (at 80.01 113.03 0)
+    (property "Footprint" "TeenieWeenieLibrary:POT_PTV09A-4025U-B104" (at 80.01 113.03 0)
       (effects (font (size 1.27 1.27)) hide)
     )
@@
       (effects (font (size 1.27 1.27)) (justify right) hide)
     )
-    (property "Footprint" "" (at 22.86 74.93 0)
+    (property "Footprint" "TeenieWeenieLibrary:POT_PTV09A-4025U-B104" (at 22.86 74.93 0)
       (effects (font (size 1.27 1.27)) hide)
     )
@@
       (effects (font (size 1.27 1.27)) (justify right) hide)
     )
-    (property "Footprint" "" (at 80.01 74.93 0)
+    (property "Footprint" "TeenieWeenieLibrary:POT_PTV09A-4025U-B104" (at 80.01 74.93 0)
       (effects (font (size 1.27 1.27)) hide)
     )
@@
       (effects (font (size 1.27 1.27)) (justify right) hide)
     )
-    (property "Footprint" "" (at 41.91 113.03 0)
-      (effects (font (size 1.27 1.27)) hide)
-    )
+    (property "Footprint" "TeenieWeenieLibrary:POT_PTV09A-4025U-B104" (at 41.91 113.03 0)
+      (effects (font (size 1.27 1.27)) hide)
+    )
