File: power.kicad_sch (KiCad schematic)
At the start: 18 parts, among them J1 Barrel_Jack, U12 AMS1117-3.3, U3 AMS1117-ADJ, U5 TLV74010PDQNR

Commit message: Finalized schematic
Parts:
- added TP1, TP2, TP3: TestPoint, TestPoint:TestPoint_Pad_1.5x1.5mm, symbol Connector:TestPoint
- C15, C16, C17, C18, C19, C20, C21, C23, C32, C33, C34, C45: footprint (none) -> Capacitor_SMD:C_0402_1005Metric
- J1: footprint (none) -> Connector_BarrelJack:BarrelJack_Horizontal
- R22, R23: footprint (none) -> Resistor_SMD:R_0402_1005Metric
- U12: footprint SOT_AMS_ADS -> TeenieWeenieLibrary:SOT_AMS_ADS
- U3: footprint SOT_AMS_ADS -> Connector_BarrelJack:BarrelJack_Horizontal
- U5: footprint SOT_PDQNR_TEX -> TeenieWeenieLibrary:SOT_PDQNR_TEX
Connections:
- net 1p8v is gone; now on net +1V8: C18.1, C19.1
- net +1V0: now also TP2.1
- net +1V8: now also TP1.1
- net +3.3V: now also TP3.1
- net GNDA renamed GND
Other:
- moved on the sheet: C15, C16, C17, C18, C19, C20, C21, C23, C32, C33, C34, C45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

Commit message: final final schematic:
Other:
- note added: "Tantalum Caps"
Changed lines of the file:
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@@
     (stroke (width 0) (type default))
+  )
+  (text "Tantalum Caps" (at 213.36 53.975 0)
+    (effects (font (size 1.27 1.27)) (justify left bottom))
+  )
+  (text "Tantalum Caps" (at 213.995 90.17 0)
+    (effects (font (size 1.27 1.27)) (justify left bottom))
+  )
+  (text "Tantalum Caps" (at 208.915 137.795 0)
+    (effects (font (size 1.27 1.27)) (justify left bottom))
   )
   (hierarchical_label "3p3V" (shape output) (at 213.36 41.91 0) (fields_autoplaced)

Commit message: rev1 of pcb component placement
Parts:
- removed TP1, TP2, TP3: TestPoint, TestPoint:TestPoint_Pad_1.5x1.5mm, symbol Connector:TestPoint
- U3: footprint Connector_BarrelJack:BarrelJack_Horizontal -> TeenieWeenieLibrary:SOT_AMS_ADS
Changed lines of the file:
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@@
-    (stroke (width 0) (type default))
-  )
-  (wire (pts (xy 191.77 74.93) (xy 191.77 78.74))
     (stroke (width 0) (type default))
   )
@@
     (stroke (width 0) (type default))
   )
-  (wire (pts (xy 187.96 127) (xy 187.96 130.81))
-    (stroke (width 0) (type default))
-  )
   (wire (pts (xy 113.03 78.74) (xy 124.46 78.74))
     (stroke (width 0) (type default))
@@
   )
   (wire (pts (xy 125.73 123.19) (xy 125.73 128.27))
-    (stroke (width 0) (type default))
-  )
-  (wire (pts (xy 194.31 38.1) (xy 194.31 41.91))
     (stroke (width 0) (type default))
   )
@@
       (effects (font (size 1.524 1.524)))
     )
-    (property "Footprint" "Connector_BarrelJack:BarrelJack_Horizontal" (at 156.21 83.82 0)
+    (property "Footprint" "TeenieWeenieLibrary:SOT_AMS_ADS" (at 156.21 83.82 0)
       (effects (font (size 1.27 1.27) italic) hide)
     )
@@
         (path "/58e2e2d3-cf30-4313-be51-7fb67401d242/e01203e1-17d3-4203-8a08-464c4ccfbd33"
           (reference "R23") (unit 1)
-        )
-      )
-    )
-  )
-  (symbol (lib_id "Connector:TestPoint") (at 191.77 74.93 0) (unit 1)
-    (in_bom yes) (on_board yes) (dnp no) (fields_autoplaced)
-    (property "Reference" "TP1" (at 194.31 70.358 0)
-      (effects (font (size 1.27 1.27)) (justify left))
-    )
-    (property "Value" "TestPoint" (at 194.31 72.898 0)
-      (effects (font (size 1.27 1.27)) (justify left))
-    )
-    (property "Footprint" "TestPoint:TestPoint_Pad_1.5x1.5mm" (at 196.85 74.93 0)
-      (effects (font (size 1.27 1.27)) hide)
-    )
-    (property "Datasheet" "~" (at 196.85 74.93 0)
-      (effects (font (size 1.27 1.27)) hide)
-    )
-    (pin "1")
-    (instances
-      (project "TeenieWeenie"
-        (path "/58e2e2d3-cf30-4313-be51-7fb67401d242/e01203e1-17d3-4203-8a08-464c4ccfbd33"
-          (reference "TP1") (unit 1)
         )
       )
@@
     )
   )
-  (symbol (lib_id "Connector:TestPoint") (at 194.31 38.1 0) (unit 1)
-    (in_bom yes) (on_board yes) (dnp no) (fields_autoplaced)
-    (property "Reference" "TP3" (at 196.85 33.528 0)
-      (effects (font (size 1.27 1.27)) (justify left))
-    )
-    (property "Value" "TestPoint" (at 196.85 36.068 0)
-      (effects (font (size 1.27 1.27)) (justify left))
-    )
-    (property "Footprint" "TestPoint:TestPoint_Pad_1.5x1.5mm" (at 199.39 38.1 0)
-      (effects (font (size 1.27 1.27)) hide)
-    )
-    (property "Datasheet" "~" (at 199.39 38.1 0)
-      (effects (font (size 1.27 1.27)) hide)
-    )
-    (pin "1")
-    (instances
-      (project "TeenieWeenie"
-        (path "/58e2e2d3-cf30-4313-be51-7fb67401d242/e01203e1-17d3-4203-8a08-464c4ccfbd33"
-          (reference "TP3") (unit 1)
-        )
-      )
-    )
-  )
   (symbol (lib_id "power:+1V8") (at 182.88 73.66 0) (unit 1)
     (in_bom yes) (on_board yes) (dnp no) (fields_autoplaced)
@@
         )
       )
-    )
-  )
-  (symbol (lib_id "Connector:TestPoint") (at 187.96 127 0) (unit 1)
-    (in_bom yes) (on_board yes) (dnp no) (fields_autoplaced)
-    (property "Reference" "TP2" (at 190.5 122.428 0)
-      (effects (font (size 1.27 1.27)) (justify left))
-    )
-    (property "Value" "TestPoint" (at 190.5 124.968 0)
-      (effects (font (size 1.27 1.27)) (justify left))
-    )
-    (property "Footprint" "TestPoint:TestPoint_Pad_1.5x1.5mm" (at 193.04 127 0)
-      (effects (font (size 1.27 1.27)) hide)
-    )
-    (property "Datasheet" "~" (at 193.04 127 0)
-      (effects (font (size 1.27 1.27)) hide)
-    )
-    (pin "1")
-    (instances
-      (project "TeenieWeenie"
-        (path "/58e2e2d3-cf30-4313-be51-7fb67401d242/e01203e1-17d3-4203-8a08-464c4ccfbd33"
-          (reference "TP2") (unit 1)
-        )
-      )
