File: TeenieWeenie.kicad_sch (KiCad schematic)
At the start: 0 parts

Commit message: Finalized schematic
Parts:
- added H1, H2, H3, H4: MountingHole, MountingHole:MountingHole_2.2mm_M2_DIN965, symbol Mechanical:MountingHole
Connections:
- no-connect marks 2 -> 0
Other:
- added sheet ADC (ADC.kicad_sch)
- sheet AFE ports: added AFE0_L, AFE0_R, AFE1_L, AFE1_R; removed ADCRDY_0, ADCRDY_1, AFE_L, AFE_R, SCL, SDA

Commit message: final final schematic:
Parts:
- added J2, J3, J4, J5, J6, J8: Conn_01x01, Connector_PinHeader_1.00mm:PinHeader_1x01_P1.00mm_Vertical, symbol Connector_Generic:Conn_01x01
Connections:
- new net AFE/AudioIn_L: J2.1 (Pin_1)
- new net AFE/AudioIn_R: J3.1 (Pin_1)
- new net GND: J4.1 (Pin_1), J8.1 (Pin_1)
- new net IOSwitch/AudioOut_L: J5.1 (Pin_1)
- new net IOSwitch/AudioOut_R: J6.1 (Pin_1)
Other:
- added sheet IOSwitch (IOSwitch.kicad_sch)
- sheet AFE ports: added AudioIn_L, AudioIn_R; removed none
- sheet AudioCodec ports: added AudioOut_L, AudioOut_R; removed none
- sheet MCU ports: added ~{SWCTRL}; removed none

Commit message: rev1 of pcb component placement
Parts:
- added U7: SM05T1G, TeenieWeenieLibrary:SOT-23_ONS, symbol TeenieWeenie:SM05T1G
Connections:
- net AFE/AudioIn_L: now also U7.1 (CATHODE)
- net AFE/AudioIn_R: now also U7.2 (CATHODE)
- net GND: now also U7.3 (ANODE)
Changed lines of the file:
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@@
   (junction (at 32.385 43.815) (diameter 0) (color 0 0 0 0)
   )
+  (junction (at 27.94 43.815) (diameter 0) (color 0 0 0 0)
+  )
+  (junction (at 35.56 46.99) (diameter 0) (color 0 0 0 0)
+  )
   (junction (at 146.05 83.82) (diameter 0) (color 0 0 0 0)
   )
@@
   (junction (at 38.735 46.99) (diameter 0) (color 0 0 0 0)
   )
+  (wire (pts (xy 27.94 43.815) (xy 27.94 59.055))
+    (stroke (width 0) (type default))
+  )
   (wire (pts (xy 186.69 22.86) (xy 202.565 22.86))
     (stroke (width 0) (type default))
@@
     (stroke (width 0) (type default))
   )
+  (wire (pts (xy 35.56 46.99) (xy 38.735 46.99))
+    (stroke (width 0) (type default))
+  )
   (wire (pts (xy 130.81 71.12) (xy 165.1 71.12))
     (stroke (width 0) (type default))
   )
+  (wire (pts (xy 31.75 76.835) (xy 31.75 79.375))
+    (stroke (width 0) (type default))
+  )
   (wire (pts (xy 130.81 119.38) (xy 146.05 119.38))
     (stroke (width 0) (type default))
@@
     (stroke (width 0) (type default))
   )
-  (wire (pts (xy 25.4 43.815) (xy 32.385 43.815))
+  (wire (pts (xy 25.4 43.815) (xy 27.94 43.815))
     (stroke (width 0) (type default))
   )
@@
     (stroke (width 0) (type default))
   )
+  (wire (pts (xy 35.56 46.99) (xy 35.56 59.055))
+    (stroke (width 0) (type default))
+  )
   (wire (pts (xy 143.51 46.99) (xy 130.81 46.99))
     (stroke (width 0) (type default))
@@
     (stroke (width 0) (type default))
   )
+  (wire (pts (xy 27.94 43.815) (xy 32.385 43.815))
+    (stroke (width 0) (type default))
+  )
   (wire (pts (xy 141.605 19.685) (xy 141.605 44.45))
     (stroke (width 0) (type default))
@@
     (stroke (width 0) (type default))
   )
-  (wire (pts (xy 25.4 46.99) (xy 38.735 46.99))
+  (wire (pts (xy 25.4 46.99) (xy 35.56 46.99))
     (stroke (width 0) (type default))
   )
@@
     )
   )
+  (symbol (lib_id "TeenieWeenie:SM05T1G") (at 31.75 69.215 0) (unit 1)
+    (in_bom yes) (on_board yes) (dnp no)
+    (property "Reference" "U7" (at 58.42 61.595 0)
+      (effects (font (size 1.524 1.524)) hide)
+    )
+    (property "Value" "SM05T1G" (at 57.15 61.595 0)
+      (effects (font (size 1.524 1.524)) hide)
+    )
+    (property "Footprint" "TeenieWeenieLibrary:SOT-23_ONS" (at 57.15 78.105 0)
+      (effects (font (size 1.27 1.27) italic) hide)
+    )
+    (property "Datasheet" "SM05T1G" (at 57.15 75.565 0)
+      (effects (font (size 1.27 1.27) italic) hide)
+    )
+    (pin "1")
+    (pin "2")
+    (pin "3")
+    (instances
+      (project "TeenieWeenie"
+        (path "/58e2e2d3-cf30-4313-be51-7fb67401d242/d79052ad-b30d-48cb-904a-b15d582d373d"
+          (reference "U7") (unit 1)
+        )
+        (path "/58e2e2d3-cf30-4313-be51-7fb67401d242"
+          (reference "U7") (unit 1)
+        )
+      )
+    )
+  )
   (symbol (lib_id "Mechanical:MountingHole") (at 232.41 124.46 0) (unit 1)
     (in_bom yes) (on_board yes) (dnp no) (fields_autoplaced)
@@
         )
       )
+    )
+  )
+  (symbol (lib_id "power:GND") (at 31.75 79.375 0) (unit 1)
+    (in_bom yes) (on_board yes) (dnp no) (fields_autoplaced)
+    (property "Reference" "#PWR058" (at 31.75 85.725 0)
+      (effects (font (size 1.27 1.27)) hide)
+    )
+    (property "Value" "GND" (at 31.75 84.455 0)
+      (effects (font (size 1.27 1.27)))
+    )
+    (property "Footprint" "" (at 31.75 79.375 0)
+      (effects (font (size 1.27 1.27)) hide)
+    )
+    (property "Datasheet" "" (at 31.75 79.375 0)
+      (effects (font (size 1.27 1.27)) hide)
+    )
+    (pin "1")
+    (instances
+      (project "TeenieWeenie"
+        (path "/58e2e2d3-cf30-4313-be51-7fb67401d242/db217c67-4148-46d6-b5bb-bc62bff1a084"
+          (reference "#PWR058") (unit 1)
+        )
+        (path "/58e2e2d3-cf30-4313-be51-7fb67401d242/d79052ad-b30d-48cb-904a-b15d582d373d"
+          (reference "#PWR034") (unit 1)
+        )
+        (path "/58e2e2d3-cf30-4313-be51-7fb67401d242"
+          (reference "#PWR0111") (unit 1)
+        )
+        (path "/58e2e2d3-cf30-4313-be51-7fb67401d242/620606a9-8957-4afc-a718-89a87c66d877"
+          (reference "#PWR0102") (unit 1)
+        )
+      )

Commit message: routed power
Connections:
- net AFE/AudioIn_L renamed AFE/AudioL_Raw
- net AFE/AudioIn_R renamed AFE/AudioR_Raw
Other:
- sheet AFE ports: added AudioL_Raw, AudioR_Raw; removed AudioIn_L, AudioIn_R
- sheet AudioCodec ports: added AudioL_Dirty, AudioR_Dirty; removed AudioOut_L, AudioOut_R
Changed lines of the file:
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@@
       (effects (font (size 1.27 1.27)) (justify right))
     )
-    (pin "AudioIn_L" input (at 41.91 44.45 180)
+    (pin "AudioL_Raw" input (at 41.91 44.45 180)
       (effects (font (size 1.27 1.27)) (justify left))
     )
-    (pin "AudioIn_R" input (at 41.91 46.99 180)
+    (pin "AudioR_Raw" input (at 41.91 46.99 180)
       (effects (font (size 1.27 1.27)) (justify left))
     )
@@
       (effects (font (size 1.27 1.27)) (justify right))
     )
-    (pin "AudioOut_L" output (at 130.81 44.45 0)
+    (pin "AudioL_Dirty" output (at 130.81 44.45 0)
       (effects (font (size 1.27 1.27)) (justify right))
     )
-    (pin "AudioOut_R" output (at 130.81 46.99 0)
+    (pin "AudioR_Dirty" output (at 130.81 46.99 0)
       (effects (font (size 1.27 1.27)) (justify right))
     )
